File: teensy_32_carrier/teensy_32_carrier.kicad_pcb (KiCad board)
At the start: 2 copper layers, 38.1 x 50.8 mm, 18 parts, among them U1 TEENSY_3

Commit message: first revision of teensy 3.2 carrier hat
Parts:
- removed D14: D14, teensy:SIP-3
- removed D15: D15, teensy:SIP-3
- removed D16: D16, teensy:SIP-3
- removed D21: D21, teensy:SIP-3
- removed D22: D22, teensy:SIP-3
- removed D23: D23, teensy:SIP-3
- removed LED3: D3, LEDs:LED-3MM
- removed LED4: D4, LEDs:LED-3MM
- removed R1, R2: 220R, Resistors_ThroughHole:Resistor_Horizontal_RM7mm
- removed RCV1: RCV1, teensy:SIP-3
- removed REF** (x4): MountingHole_3mm, Mounting_Holes:MountingHole_3mm
- removed RX1: RX1, teensy:SIP-3
- removed SVO1: SVO1, teensy:SIP-3
- removed U1: TEENSY_3, teensy:TEENSY_3
Routing:
- net Net-(RX1-Pad2): track 34.5 -> 0.00 mm
- net /D4: track 29.5 -> 0.00 mm
- net Net-(RX1-Pad1): track 28.6 -> 0.00 mm
- net /D3: track 20.8 -> 0.00 mm, vias 2 -> 0
- net Net-(D23-Pad1): track 9.20 -> 0.00 mm
- net Net-(D21-Pad1): track 9.20 -> 0.00 mm
- net Net-(D22-Pad1): track 9.20 -> 0.00 mm
- net Net-(D16-Pad1): track 8.15 -> 0.00 mm
- net Net-(D15-Pad1): track 8.15 -> 0.00 mm
- net Net-(D14-Pad1): track 8.15 -> 0.00 mm
- net Net-(LED4-Pad2): track 7.62 -> 0.00 mm
- net Net-(LED3-Pad2): track 7.62 -> 0.00 mm
- net +6V: track 7.62 -> 0.00 mm
- net +5V: track 7.62 -> 0.00 mm
- removed copper zone on B.Cu, net GND
- removed copper zone on F.Cu, net VCC
Other:
- board outline removed
- net class Default: trace_width 0.35 -> 0.25; via_dia 0.7 -> 0.6; via_drill 0.5 -> 0.4
- rule pad_to_mask_clearance: 0.2 -> 0
- board text removed: "CONTROLS"
- board text removed: "G"
- board text removed: "Onyx Robots Teensy 3.2 Servo Interface github.com/jwatte/donkey_racing v1.0 2017-08-14"
- board text removed: "RECEIVER"
- board text removed: "Vin"

Commit message: first batch of layout
Parts:
- added C1: MF-CAP-0603-0.1UF, MF_Passives:MF_Passives-C0603, B.Cu at (115.5, 80.5)
- added C10: 311-2054-1-ND, MF_Passives:MF_Passives-C1210, B.Cu at (83.4, 76.7)
- added C11: MF-CAP-10MM-470uF, MF_Passives:MF_Passives-CP10MM, F.Cu at (81.7, 73.2)
- added C12: 311-2054-1-ND, MF_Passives:MF_Passives-C1210, B.Cu at (88.5, 95.0)
- added C3: MF-CAP-6.3MM-100uF, MF_Passives:MF_Passives-CP6.3MM, F.Cu at (93.0, 105.5)
- added C4: MF-CAP-6.3MM-100uF, MF_Passives:MF_Passives-CP6.3MM, F.Cu at (87.0, 96.5)
- added C5: MF-CAP-0402-0.01uF, MF_Passives:MF_Passives-C0402, B.Cu at (94.0, 85.0)
- added C6: MF-CAP-0603-0.1UF, MF_Passives:MF_Passives-C0603, B.Cu at (94.5, 86.5)
- added C7: 311-2054-1-ND, MF_Passives:MF_Passives-C1210, B.Cu at (83.4, 80.3)
- added C8: 311-2054-1-ND, MF_Passives:MF_Passives-C1210, B.Cu at (83.4, 73.2)
- added C9: 311-2054-1-ND, MF_Passives:MF_Passives-C1210, B.Cu at (83.4, 69.6)
- added D1: MF-LED-3228-RGB, MF_LEDs:MF_LEDs-PLCC4, F.Cu at (95.5, 70.5)
- added D2: MM3Z15VT1GOSCT-ND, Diodes_SMD:SOD-323, B.Cu at (89.0, 106.0)
- added D3: 1655-1752-1-ND, teensy:TO-277B, F.Cu at (91.1, 73.3)
- added D6: 1727-5317-1-ND, teensy:SOD-128, F.Cu at (94.0, 99.0)
- added J1: CON_01X03_PTH_2.54MM, MF_Connectors:MF_Connectors-PTH_2.54MM_01X03, F.Cu at (97.5, 81.5)
- added J10: CJ, teensy:CJ-2, B.Cu at (132.0, 85.0)
- added J11: CJ, teensy:CJ-2, B.Cu at (132.0, 82.4)
- added J12: CJ, teensy:CJ-2, B.Cu at (132.0, 79.7)
- added J13: CJ, teensy:CJ-2, B.Cu at (132.0, 77.0)
- added J14: CJ, teensy:CJ-2, B.Cu at (95.5, 111.5)
- added J2: CON_01X08_PTH_2.54MM, MF_Connectors:MF_Connectors-PTH_2.54MM_01X08, F.Cu at (111.5, 104.0)
- added J3: CON_01X06_PTH_2.54MM, MF_Connectors:MF_Connectors-PTH_2.54MM_01X06, F.Cu at (102.0, 80.0)
- added J4: CON_01X04_PTH_2.54MM, MF_Connectors:MF_Connectors-PTH_2.54MM_01X04, F.Cu at (134.0, 96.5)
- added J5: CON_01X03_PTH_2.54MM, MF_Connectors:MF_Connectors-PTH_2.54MM_01X03, F.Cu at (99.5, 96.5)
- added J6: CON_01X03_PTH_2.54MM, MF_Connectors:MF_Connectors-PTH_2.54MM_01X03, F.Cu at (126.5, 96.5)
- added J7: CON_01X08_PTH_2.54MM, MF_Connectors:MF_Connectors-PTH_2.54MM_01X08, F.Cu at (109.1, 67.9)
- added J8: CON_01X05_PTH_2.54MM, MF_Connectors:MF_Connectors-PTH_2.54MM_01X05, F.Cu at (127.4, 67.9)
- added J9: CON_01X05_PTH_2.54MM, MF_Connectors:MF_Connectors-PTH_2.54MM_01X05, F.Cu at (132.5, 104.0)
- added L1: SRP1238A-8R2MCT-ND, teensy:BOURNS_SRP1238A, F.Cu at (83.1, 85.1)
- added P1: S9200-ND, teensy:RPI_BOTTOM_NOLABELS, B.Cu at (107.5, 63.5)
- added P2: CONN_01X02, teensy:SCREW-3.5MM, F.Cu at (87.6, 113.7)
- added P3: CONN_01X02, teensy:SCREW-3.5MM, F.Cu at (78.1, 104.0)
- added Q1: STL62P3LLH6, teensy:POWERFLAT_5x6, F.Cu at (86.0, 106.0)
- added R1: MF-RES-0603-604K, MF_Passives:MF_Passives-R0603, B.Cu at (118.5, 82.0)
- added R10: 311-56.0KLRCT-ND, MF_Passives:MF_Passives-R0402, B.Cu at (97.5, 92.5)
- added R11: MF-RES-0402-100K, MF_Passives:MF_Passives-R0402, B.Cu at (82.5, 84.5)
- added R12: 311-17.4KLRCT-ND, MF_Passives:MF_Passives-R0402, B.Cu at (85.1, 84.5)
- added R13: MF-RES-0402-2K, MF_Passives:MF_Passives-R0402, B.Cu at (123.0, 76.0)
- added R14: MF-RES-0402-2K, MF_Passives:MF_Passives-R0402, B.Cu at (124.5, 76.0)
- added R15: MF-RES-0402-100K, MF_Passives:MF_Passives-R0402, B.Cu at (96.8, 98.8)
- added R16: 311-14.0KLRCT-ND, MF_Passives:MF_Passives-R0402, B.Cu at (96.8, 96.1)
- added R17: MF-RES-0402-10K, MF_Passives:MF_Passives-R0402, B.Cu at (98.0, 108.0)
- added R2: MF-RES-0603-100K, MF_Passives:MF_Passives-R0603, B.Cu at (115.5, 82.0)
- added R3: MF-RES-0402-220, MF_Passives:MF_Passives-R0402, B.Cu at (99.0, 71.0)
- added R4: MF-RES-0402-60.4, MF_Passives:MF_Passives-R0402, B.Cu at (99.0, 74.0)
- added R5: MF-RES-0402-22, MF_Passives:MF_Passives-R0402, B.Cu at (99.0, 72.5)
- added R6: MF-RES-0402-10K, MF_Passives:MF_Passives-R0402, B.Cu at (100.0, 104.5)
- added R7: MF-RES-0402-10K, MF_Passives:MF_Passives-R0402, B.Cu at (105.5, 112.5)
- added R8: MF-RES-0402-4.7K, MF_Passives:MF_Passives-R0402, B.Cu at (110.0, 107.0)
- added R9: MF-RES-0402-470, MF_Passives:MF_Passives-R0402, B.Cu at (106.5, 110.0)
- added RA1: MF-RES-ARRAY-1K, MF_Passives:MF_Passives-RA1206, B.Cu at (126.5, 82.0)
- added REF**: MountingHole_2-7mm, Mounting_Holes:MountingHole_2-7mm, F.Cu at (78.5, 113.0)
- added REF**: MountingHole_2-7mm, Mounting_Holes:MountingHole_2-7mm, F.Cu at (136.5, 113.0)
- added REF**: MountingHole_2-7mm, Mounting_Holes:MountingHole_2-7mm, F.Cu at (136.5, 63.5)
- added REF**: MountingHole_2-7mm, Mounting_Holes:MountingHole_2-7mm, F.Cu at (78.5, 63.5)
- added SW1: TACT_6MM, MF_Switches:MF_Switches-TACT6MM, F.Cu at (129.4, 111.0)
- added SW2: TACT_6MM, MF_Switches:MF_Switches-TACT6MM, F.Cu at (118.5, 111.0)
- added SW3: MF-SW-TACT-6MM, MF_Switches:MF_Switches-TACT6MM, F.Cu at (110.0, 111.0)
- added SW4: MF-SW-TACT-6MM, MF_Switches:MF_Switches-TACT6MM, F.Cu at (100.5, 111.0)
- added U1: ED3052-5-ND, teensy:TEENSY_3, F.Cu at (121.9, 80.4)
- added U2: SAM10855-ND, teensy:CONN_03x08, F.Cu at (110.5, 96.5)
- added U3: MF-DSC-SOT223-BSS138, MF_Discrete_Semiconductor:MF_Discrete_Semiconductor-SOT-23-3, B.Cu at (101.0, 108.0)
- added U4: MF-DSC-SOT223-BSS138, MF_Discrete_Semiconductor:MF_Discrete_Semiconductor-SOT-23-3, B.Cu at (102.0, 112.5)
- added U5: LMR14050, teensy:POWERPAD-8, F.Cu at (94.5, 90.8)
Other:
- board outline added: 65 x 56.5 mm
- board text added: "Cut Here"
- board text added: "RXD"
- board text added: "SCL"
- board text added: "SDA"
- board text added: "Stay On"
- board text added: "TXD"

Commit message: set up design rules
Parts:
- P2, P3: value CONN_01X02 -> A98159-ND
Other:
- copper layers 2 -> 4
- rule trace_min: 0.2 -> 0.13
- rule via_min_drill: 0.3 -> 0.305
- rule via_min_size: 0.4 -> 0.465
Changed lines of the file:
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@@
   (page A4)
   (layers
-    (0 F.Cu signal)
+    (0 F.Cu power)
+    (1 In1.Cu signal)
+    (2 In2.Cu signal)
     (31 B.Cu signal)
     (32 B.Adhes user)
@@
     (46 B.CrtYd user)
     (47 F.CrtYd user)
-    (48 B.Fab user hide)
-    (49 F.Fab user hide)
+    (48 B.Fab user)
+    (49 F.Fab user)
   )
   (setup
     (last_trace_width 0.25)
+    (user_trace_width 0.5)
+    (user_trace_width 1)
+    (user_trace_width 1.5)
+    (user_trace_width 2.3)
     (trace_clearance 0.2)
     (zone_clearance 0.508)
     (zone_45_only no)
-    (trace_min 0.2)
+    (trace_min 0.13)
     (segment_width 0.2)
     (edge_width 0.2)
     (via_size 0.6)
     (via_drill 0.4)
-    (via_min_size 0.4)
-    (via_min_drill 0.3)
-    (uvia_size 0.3)
-    (uvia_drill 0.1)
+    (via_min_size 0.465)
+    (via_min_drill 0.305)
+    (user_via 0.85 0.6)
+    (user_via 1.25 1)
+    (uvia_size 0.51)
+    (uvia_drill 0.13)
     (uvias_allowed no)
-    (uvia_min_size 0.2)
+    (uvia_min_size 0.18)
     (uvia_min_drill 0.1)
     (pcb_text_width 0.3)
@@
     (via_dia 0.6)
     (via_drill 0.4)
-    (uvia_dia 0.3)
-    (uvia_drill 0.1)
+    (uvia_dia 0.51)
+    (uvia_drill 0.13)
     (add_net +2V5)
     (add_net +3V3)
@@
       (effects (font (size 1 1) (thickness 0.15)))
     )
-    (fp_text value CONN_01X02 (at 0 -6.35 270) (layer F.Fab)
+    (fp_text value A98159-ND (at 0 -6.35 270) (layer F.Fab)
       (effects (font (size 1 1) (thickness 0.15)))
     )
@@
       (effects (font (size 1 1) (thickness 0.15)))
     )
-    (fp_text value CONN_01X02 (at 0 -6.35) (layer F.Fab)
+    (fp_text value A98159-ND (at 0 -6.35) (layer F.Fab)
       (effects (font (size 1 1) (thickness 0.15)))
     )
