File: teensy_32_carrier/teensy_32_carrier.sch (KiCad schematic (older format))
At the start: 14 parts, among them U1 TEENSY_3

Commit message: first revision of teensy 3.2 carrier hat
Parts:
- removed D14: D14, teensy:SIP-3, symbol CONN_01X03
- removed D15: D15, teensy:SIP-3, symbol CONN_01X03
- removed D16: D16, teensy:SIP-3, symbol CONN_01X03
- removed D21: D21, teensy:SIP-3, symbol CONN_01X03
- removed D22: D22, teensy:SIP-3, symbol CONN_01X03
- removed D23: D23, teensy:SIP-3, symbol CONN_01X03
- removed LED3: D3, LEDs:LED-3MM, symbol Led_Small
- removed LED4: D4, LEDs:LED-3MM, symbol Led_Small
- removed R1, R2: 220R, Resistors_ThroughHole:Resistor_Horizontal_RM7mm, symbol R
- removed RCV1: RCV1, teensy:SIP-3, symbol CONN_01X03
- removed RX1: RX1, teensy:SIP-3, symbol CONN_01X03
- removed SVO1: SVO1, teensy:SIP-3, symbol CONN_01X03
- added BATT1: 952-1735-1-ND, MF_Connectors:MF_Connectors-BAT-HLD-001, symbol BATTERY_BAT-HLD-001
- added C1: MF-CAP-0603-0.1UF, MF_Passives_C0603, symbol CAPACITOR_NP_0603
- added C13, C2: MF-CAP-0603-0.1UF, MF_Passives:MF_Passives-C0603, symbol CAPACITOR_NP_0603
- added D1: MF-LED-3228-RGB, MF_LEDs:MF_LEDs-PLCC4, symbol LED_RGB_CA_PLCC4
- added D4, D5: MF-DIO-SOD123-BAT42, MF_Discrete_Semiconductor:MF_Discrete_Semiconductor-SOD-123, symbol DIODES_SOD-123
- added IC1: AT24CS32-STUM, MF_IC_Power:MF_IC_Power-SOT-23-5, symbol AT24CS32-STUM
- added J1, J5, J6: CON_01X03_PTH_2.54MM, MF_Connectors:MF_Connectors-PTH_2.54MM_01X03, symbol CON_01X03_PTH_2.54MM
- added J2, J7: CON_01X08_PTH_2.54MM, MF_Connectors:MF_Connectors-PTH_2.54MM_01X08, symbol CON_01X08_PTH_2.54MM
- added J3: CON_01X06_PTH_2.54MM, MF_Connectors:MF_Connectors-PTH_2.54MM_01X06, symbol CON_01X06_PTH_2.54MM
- added J4: CON_01X04_PTH_2.54MM, MF_Connectors:MF_Connectors-PTH_2.54MM_01X04, symbol CON_01X04_PTH_2.54MM
- added J8: CON_01X05_PTH_2.54MM, MF_Connectors:MF_Connectors-PTH_2.54MM_01X05, symbol CON_01X05_PTH_2.54MM
- added P1: CONN_02X20, teensy:RPI_BOTTOM, symbol CONN_02X20
- added R1: MF-RES-0402-825K, MF_Passives:MF_Passives-R0402, symbol RESISTOR_0402
- added R13, R14: MF-RES-0402-2K, MF_Passives:MF_Passives-R0402, symbol RESISTOR_0402
- added R2: MF-RES-0402-255K, MF_Passives:MF_Passives-R0402, symbol RESISTOR_0402
- added R3: MF-RES-0402-220, MF_Passives:MF_Passives-R0402, symbol RESISTOR_0402
- added R4: MF-RES-0402-60.4, MF_Passives:MF_Passives-R0402, symbol RESISTOR_0402
- added R5: MF-RES-0402-22, MF_Passives:MF_Passives-R0402, symbol RESISTOR_0402
- added RA1: MF-RES-ARRAY-1K, MF_Passives_RA1206, symbol RESISTOR_QUAD_ARRAY_A1206
- added SW1, SW2: TACT_6MM, MF_Switches:MF_Switches-TACT6MM, symbol TACT_6MM
- added U2: SAM10855-ND, teensy:CONN_03x08, symbol CONN_03x08
- added U6: PCF8563TS/5, teensy:TSSOP-8, symbol PCF8563
- added Y1: 728-1076-1-ND, teensy:SC-20S, symbol Crystal_Small
Connections:
- net labels added: +2V5, +3V3, +5VP, +BATT, D10, D13, D15, D17, D20, D21, D22, D23, D5, D6, D9, DIN, DOUT, PWRON, RX1, RX3, R_12, R_13, R_16, R_17, R_18, R_19, R_20, R_21, R_22, R_23, R_24, R_25, R_26, R_27, R_4, R_5, R_6, R_CE0, R_CE1, R_ID_SC, R_ID_SD, R_MISO, R_MOSI, R_RXD, R_SCK, R_SCL, R_SDA, R_TXD, SCK/D14, SCL, SDA, TX1, TX3, VSENSE
- net labels removed: +6V, VCC
- wire segments 45 -> 219
Other:
- note added: "Buttons"
- note added: "Hat EEPROM"
- note added: "I/O Power Select"
- note added: "If someone configures pins to drive into \neach other, don't burn out the ports, so \nadd a current limiting resistor on the serial\nport."
- note added: "RPi Header"
- note added: "RPi I2C"
- note added: "RPi LED"
- note added: "RPi SPI"
- note added: "RTC"
- note added: "Raspberry Pi 3V is not 2.5V, but I need\nto keep it separate from Teensy 3.3V, and \nboth "3V3" and "3.3V" rails tie together, \nand I don't yet know how to define a new \n3V3B rail. To clean up!"
- note added: "Receiver In"
- note added: "Receiver Power Select"
- note added: "Servo Power Select"
- note added: "Servo/ESC Out"
- note added: "T3 I2C"
- note added: "T3 SPI"
- note added: "T3 Serial3"

Commit message: first batch of layout
Parts:
- removed BATT1: 952-1735-1-ND, MF_Connectors:MF_Connectors-BAT-HLD-001, symbol BATTERY_BAT-HLD-001
- removed C13, C2: MF-CAP-0603-0.1UF, MF_Passives:MF_Passives-C0603, symbol CAPACITOR_NP_0603
- removed D4, D5: MF-DIO-SOD123-BAT42, MF_Discrete_Semiconductor:MF_Discrete_Semiconductor-SOD-123, symbol DIODES_SOD-123
- removed IC1: AT24CS32-STUM, MF_IC_Power:MF_IC_Power-SOT-23-5, symbol AT24CS32-STUM
- removed U6: PCF8563TS/5, teensy:TSSOP-8, symbol PCF8563
- removed Y1: 728-1076-1-ND, teensy:SC-20S, symbol Crystal_Small
- added J10, J11, J12, J13: CJ, teensy:CJ-2, symbol CJ
- C1: footprint MF_Passives_C0603 -> MF_Passives:MF_Passives-C0603
- J8: LABEL01 SDA -> GND; LABEL02 SCL -> +3V3; LABEL04 +3.3V -> SCL; LABEL05 GND -> SDA
- P1: value CONN_02X20 -> S9200-ND; footprint teensy:RPI_BOTTOM -> teensy:RPI_BOTTOM_NOLABELS
- R1: value MF-RES-0402-825K -> MF-RES-0603-604K; footprint MF_Passives:MF_Passives-R0402 -> MF_Passives:MF_Passives-R0603
- R2: value MF-RES-0402-255K -> MF-RES-0603-100K; footprint MF_Passives:MF_Passives-R0402 -> MF_Passives:MF_Passives-R0603
- RA1: footprint MF_Passives_RA1206 -> MF_Passives:MF_Passives-RA1206
- U1: value TEENSY_3 -> ED3052-5-ND
Connections:
- wire segments 219 -> 229
Other:
- note added: "If someone configures pins to drive into \neach other, don't burn out the ports, so \nadd a current limiting resistor on the pins"
- note removed: "Hat EEPROM"
- note removed: "If someone configures pins to drive into \neach other, don't burn out the ports, so \nadd a current limiting resistor on the serial\nport."
- note removed: "RTC"
- moved on the sheet: C1, D1, J1, J3, J5, J6, J7, J8, P1, R1, R13, R14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

Commit message: Choose a part for screw terminals.
Connections:
- wire segments 229 -> 195
Changed lines of the file:
@@
 	3850 5850 3750 5850
 Wire Wire Line
-	3750 5850 3750 5950
-Wire Wire Line
-	3750 5950 3750 6050
-Wire Wire Line
-	3750 6050 3750 6150
-Wire Wire Line
-	3750 6150 3750 6250
-Wire Wire Line
-	3750 6250 3750 6350
-Wire Wire Line
-	3750 6350 3750 6450
-Wire Wire Line
-	3750 6450 3750 6550
-Wire Wire Line
-	3750 6550 3750 6800
+	3750 5850 3750 6800
 Wire Wire Line
 	3850 6550 3750 6550
@@
 	3650 5850 3550 5850
 Wire Wire Line
-	3550 5350 3550 5850
-Wire Wire Line
-	3550 5850 3550 5950
-Wire Wire Line
-	3550 5950 3550 6050
-Wire Wire Line
-	3550 6050 3550 6150
+	3550 5350 3550 6150
 Wire Wire Line
 	3550 5950 3650 5950
@@
 	3650 6250 3550 6250
 Wire Wire Line
-	3550 6250 3550 6350
-Wire Wire Line
-	3550 6350 3550 6450
-Wire Wire Line
-	3550 6450 3550 6550
-Wire Wire Line
-	3550 6550 3550 7400
+	3550 6250 3550 7400
 Wire Wire Line
 	3650 6350 3550 6350
@@
 $EndComp
 Wire Wire Line
-	1100 1250 1350 1250
-Wire Wire Line
-	1350 1250 1450 1250
+	1100 1250 1450 1250
 Wire Wire Line
 	1100 1250 1100 950
@@
 TX3
 Wire Wire Line
-	1050 3750 1050 4350
-Wire Wire Line
-	1050 4350 1050 4350
+	1050 3750 1050 4550
 $Comp
 L RESISTOR_0402 R2
@@
 $EndComp
 Wire Wire Line
-	1050 3100 1050 3200
-Wire Wire Line
-	1050 3200 1050 3350
+	1050 3100 1050 3350
 $Comp
 L RESISTOR_0402 R1
@@
 Connection ~ 1050 4350
 Wire Wire Line
-	700  3200 1050 3200
-Wire Wire Line
-	1050 3200 1650 3200
+	700  3200 1650 3200
 Wire Wire Line
 	700  3200 700  3900
@@
 	8800 2300 9350 2300
 Wire Wire Line
-	8800 850  8800 950
-Wire Wire Line
-	8800 950  8800 2300
-Wire Wire Line
-	8800 2300 8800 3100
+	8800 850  8800 3100
 Wire Wire Line
 	9100 2400 9350 2400
@@
 	9100 2600 9350 2600
 Wire Wire Line
-	8900 2700 8900 3500
-Wire Wire Line
-	8900 3500 8900 4200
-Wire Wire Line
-	8900 4200 8900 4500
+	8900 2700 8900 4500
 Wire Wire Line
 	8900 2700 9350 2700
@@
 Connection ~ 8900 4200
 Wire Wire Line
-	10450 2050 10450 2300
-Wire Wire Line
-	10450 2300 10450 2400
+	10450 2050 10450 2400
 Wire Wire Line
 	10450 2300 9850 2300
@@
 	9850 2500 10350 2500
 Wire Wire Line
-	10350 2500 10350 2900
-Wire Wire Line
-	10350 2900 10350 3200
-Wire Wire Line
-	10350 3200 10350 3700
-Wire Wire Line
-	10350 3700 10350 3900
-Wire Wire Line
-	10350 3900 10350 4500
+	10350 2500 10350 4500
 $Comp
 L GND #PWR018
@@
 	1    0    0    -1
 $EndComp
-Wire Wire Line
-	1050 4350 1050 4550
 $Comp
 L GND #PWR021
@@
 $EndComp
 Wire Wire Line
-	7750 950  8450 950
-Wire Wire Line
-	8450 950  8800 950
+	7750 950  8800 950
 Connection ~ 8450 950
 Wire Wire Line
@@
 	5800 1150 5650 1150
 Wire Wire Line
-	5650 1150 5650 1700
-Wire Wire Line
-	5650 1700 5650 2050
+	5650 1150 5650 2050
 Wire Wire Line
 	5800 1700 5650 1700
@@
 R_SDA
 Wire Wire Line
-	7750 4300 7750 4500
-Wire Wire Line
-	7750 4500 7750 5450
-Wire Wire Line
-	6650 5150 7450 5150
-Wire Wire Line
-	7450 5150 7850 5150
-Wire Wire Line
-	7150 5250 7600 5250
-Wire Wire Line
-	7600 5250 7850 5250
+	7750 4300 7750 5450
+Wire Wire Line
+	6650 5150 7850 5150
+Wire Wire Line
+	7150 5250 7850 5250
 $Comp
 L RESISTOR_0402 R13
@@
 $EndComp
 Wire Wire Line
-	7450 4500 7600 4500
-Wire Wire Line
-	7600 4500 7750 4500
+	7450 4500 7750 4500
 Connection ~ 8800 950
 Wire Wire Line
 	8450 950  8450 850
 Wire Wire Line
-	1800 4350 1050 4350
+	700  4350 1800 4350
 NoConn ~ 1800 3950
 Wire Wire Line
 	700  4350 700  4100
-Wire Wire Line
-	700  4350 1050 4350
-Connection ~ 1050 4350
 $EndSCHEMATC

Commit message: version 0.1 ready to test upload
Changed lines of the file:
@@
 	5150 2700 5550 2700
 Text Label 5250 2700 0    60   ~ 0
-R_26
+R_17
 $Comp
 L TACT_6MM SW1
@@
 $EndComp
 NoConn ~ 10150 2800
-NoConn ~ 9100 2800
-NoConn ~ 9100 2900
 NoConn ~ 9100 3000
 NoConn ~ 10150 3000
@@
 Wire Wire Line
 	700  4350 700  4100
+NoConn ~ 9100 2900
+NoConn ~ 9100 4100
 $EndSCHEMATC

Commit message: trying to fit an RTC and the Hat EEPROM, but no.
Parts:
- J1, J5, J6: value CON_01X03_PTH_2.54MM -> MF-CON-2.54mm-01x03
- J2, J7: value CON_01X08_PTH_2.54MM -> MF-CON-2.54mm-01x08
- J3: value CON_01X06_PTH_2.54MM -> MF-CON-2.54mm-01x06
- J4: value CON_01X04_PTH_2.54MM -> MF-CON-2.54mm-01x04
- J8: value CON_01X05_PTH_2.54MM -> MF-CON-2.54mm-01x05
Other:
- note added: "If someone configures pins to drive into \neach other, don't burn out the ports, so \nhere's a current limiting resistor on the pins"
- note added: "Raspberry Pi 3V is not 2.5V, but I need\nto keep it separate from Teensy 3.3V, and \nboth "3V3" and "3.3V" rails tie together, \nand I don't yet know how to define a new \n3V3B rail in KiCad. To clean up!"
- note removed: "If someone configures pins to drive into \neach other, don't burn out the ports, so \nadd a current limiting resistor on the pins"
- note removed: "Raspberry Pi 3V is not 2.5V, but I need\nto keep it separate from Teensy 3.3V, and \nboth "3V3" and "3.3V" rails tie together, \nand I don't yet know how to define a new \n3V3B rail. To clean up!"
- moved on the sheet: D1, J10, J11, J12, J13, J8, R13, R14, R3, R4, R5, RA1A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

Commit message: version 2 macrofab project
Connections:
- wire segments 195 -> 199
- no-connect marks 16 -> 14
Changed lines of the file:
@@
 $Descr A4 11693 8268
 encoding utf-8
-Sheet 1 2
+Sheet 1 3
 Title ""
 Date ""
@@
 	1    0    0    -1
 $EndComp
-Wire Wire Line
-	9100 3600 9350 3600
 Wire Wire Line
 	9100 3700 9350 3700
@@
 Text Notes 8950 1650 0    59   ~ 0
 Raspberry Pi 3V is not 2.5V, but I need\nto keep it separate from Teensy 3.3V, and \nboth "3V3" and "3.3V" rails tie together, \nand I don't yet know how to define a new \n3V3B rail in KiCad. To clean up!
-Text Notes 5600 4950 0    39   ~ 0
+Text Notes 5500 3550 0    39   ~ 0
 If someone configures pins to drive into \neach other, don't burn out the ports, so \nhere's a current limiting resistor on the pins
 Wire Wire Line
@@
 Wire Wire Line
 	6900 3850 6900 4000
-NoConn ~ 9100 3600
-NoConn ~ 10150 3600
+$Sheet
+S 6550 5150 1200 1150
+U 59B9BC3F
+F0 "I2C Stuff" 60
+F1 "i2cstuff.sch" 60
+F2 "R_ID_SD" I R 7750 6100 60
+F3 "R_ID_SC" I R 7750 5950 60
+F4 "R_SDA" I R 7750 5600 60
+F5 "R_SCL" I R 7750 5450 60
+$EndSheet
+Wire Wire Line
+	7750 5450 8450 5450
+Wire Wire Line
+	7750 5600 8450 5600
+Wire Wire Line
+	7750 5950 8450 5950
+Wire Wire Line
+	7750 6100 8450 6100
+Wire Wire Line
+	9100 3600 9350 3600
+Text Label 7900 5950 0    60   ~ 0
+R_ID_SC
+Text Label 7900 6100 0    60   ~ 0
+R_ID_SD
+Text Label 7900 5450 0    60   ~ 0
+R_SCL
+Text Label 7900 5600 0    60   ~ 0
+R_SDA
 $EndSCHEMATC

Commit message: carrier update
Parts:
- C1: value MF-CAP-0603-0.1UF -> MF-CAP-0603-0.1uF
- SW1, SW2: value TACT_6MM -> MF-SW-TACT-6MM
Changed lines of the file:
@@
 P 700 4000
 F 0 "C1" V 650 4100 45  0000 L BNN
-F 1 "MF-CAP-0603-0.1UF" V 850 3700 45  0000 L BNN
+F 1 "MF-CAP-0603-0.1uF" V 850 3700 45  0000 L BNN
 F 2 "MF_Passives:MF_Passives-C0603" H 950 3910 20  0001 C CNN
 F 3 "" H 700 4000 60  0001 C CNN
@@
 P 5900 1050
 F 0 "SW1" H 5800 1350 45  0000 L CNN
-F 1 "TACT_6MM" H 5800 1270 45  0000 L CNN
+F 1 "MF-SW-TACT-6MM" H 5800 1270 45  0000 L CNN
 F 2 "MF_Switches:MF_Switches-TACT6MM" H 5800 1210 20  0001 L CNN
 F 3 "" H 5900 1050 60  0001 C CNN
@@
 P 5900 1600
 F 0 "SW2" H 5800 1900 45  0000 L CNN
-F 1 "TACT_6MM" H 5800 1820 45  0000 L CNN
+F 1 "MF-SW-TACT-6MM" H 5800 1820 45  0000 L CNN
 F 2 "MF_Switches:MF_Switches-TACT6MM" H 5800 1760 20  0001 L CNN
 F 3 "" H 5900 1600 60  0001 C CNN
