File: teensy_32_v2/_saved_power.sch (KiCad schematic (older format))
At the start: 31 parts, among them J1 277-1667-ND, J2 277-1667-ND, Q1 STL62P3LLH6, U2 MF-DSC-SOT233-BSS138, U3 DS7257G

Commit message: progress on new hat
Parts:
- U3: footprint (none) -> teensy:SOP-8
Changed lines of the file:
@@
 $EndComp
 Wire Wire Line
-	1200 2400 1650 2400
-Wire Wire Line
-	1650 2400 2600 2400
-Wire Wire Line
-	2600 2400 3100 2400
-Wire Wire Line
-	3100 2400 3300 2400
+	1200 2400 3300 2400
 Wire Wire Line
 	2650 2400 3100 2400
 Wire Wire Line
-	3700 2400 4800 2400
-Wire Wire Line
-	4800 2400 6550 2400
-Wire Wire Line
-	6550 2400 10300 2400
+	3700 2400 10300 2400
 Wire Wire Line
 	1200 2500 1450 2500
 Wire Wire Line
-	1450 2500 1450 3850
-Wire Wire Line
-	1450 3850 1450 4350
+	1450 2500 1450 4350
 Wire Wire Line
 	3100 2400 3100 2600
@@
 	3100 3000 3100 3250
 Wire Wire Line
-	2600 3250 3100 3250
-Wire Wire Line
-	3100 3250 3500 3250
-Wire Wire Line
-	3500 2700 3500 3250
-Wire Wire Line
-	3500 3250 3500 3350
-Wire Wire Line
-	3500 3750 3500 3900
-Wire Wire Line
-	3500 3900 3500 4050
+	2600 3250 3500 3250
+Wire Wire Line
+	3500 2700 3500 3350
+Wire Wire Line
+	3500 3750 3500 4050
 Connection ~ 3500 3250
 Wire Wire Line
-	3500 4650 3500 5150
-Wire Wire Line
-	3500 5150 3500 5400
-Wire Wire Line
-	3100 5150 3500 5150
-Wire Wire Line
-	3500 5150 4000 5150
+	3500 4650 3500 5400
+Wire Wire Line
+	3100 5150 4000 5150
 Wire Wire Line
 	4000 5150 4000 4950
 Connection ~ 3500 5150
 Wire Wire Line
-	4000 3900 4000 4350
-Wire Wire Line
-	4000 4350 4000 4550
-Wire Wire Line
-	3900 4350 4000 4350
-Wire Wire Line
-	4000 4350 4350 4350
+	4000 3900 4000 4550
+Wire Wire Line
+	3900 4350 4350 4350
 Connection ~ 4000 4350
 Wire Wire Line
@@
 	4000 3350 4000 3500
 Wire Wire Line
-	4800 1800 4800 2050
-Wire Wire Line
-	4800 2050 4800 2400
-Wire Wire Line
-	4800 2400 4800 2600
+	4800 1800 4800 2600
 Connection ~ 4800 2400
 Wire Wire Line
-	4800 3900 4800 4200
-Wire Wire Line
-	4800 4200 4800 5400
-Wire Wire Line
-	4800 3000 4800 3300
-Wire Wire Line
-	4800 3300 4800 3500
+	4800 3900 4800 5400
+Wire Wire Line
+	4800 3000 4800 3500
 Wire Wire Line
 	4800 3300 5050 3300
 Wire Wire Line
-	5050 2950 5050 3300
-Wire Wire Line
-	5050 3300 5050 3600
+	5050 2950 5050 3600
 Connection ~ 4800 3300
 Connection ~ 5050 3300
@@
 	10100 2500 10100 3100
 Wire Wire Line
-	6550 2900 6550 3050
-Wire Wire Line
-	6550 3050 6550 3400
-Wire Wire Line
-	6550 3400 6550 3750
-Wire Wire Line
-	6550 3750 6550 3950
+	6550 2900 6550 3950
 Wire Wire Line
 	4350 4350 4350 4000
@@
 	5850 3400 5450 3400
 Wire Wire Line
-	5450 3050 5450 3400
-Wire Wire Line
-	5450 3400 5450 3750
-Wire Wire Line
-	5450 3750 5450 5300
-Wire Wire Line
-	5450 5300 5450 5400
+	5450 3050 5450 5400
 Wire Wire Line
 	7550 4550 7400 4550
@@
 	7100 4350 7550 4350
 Wire Wire Line
-	8850 3850 8950 3850
-Wire Wire Line
-	8950 3850 9000 3850
+	8850 3850 9000 3850
 Wire Wire Line
 	6000 4150 6000 4750
@@
 	7100 4750 7100 4350
 Wire Wire Line
-	8850 4150 9300 4150
-Wire Wire Line
-	9300 4150 9550 4150
+	8850 4150 9550 4150
 Wire Wire Line
 	9300 4150 9300 3850
 Connection ~ 9300 4150
 Wire Wire Line
-	10650 4150 10300 4150
-Wire Wire Line
-	10300 4150 9950 4150
-Wire Wire Line
-	9950 4150 9750 4150
-Wire Wire Line
-	10650 3400 10650 3600
-Wire Wire Line
-	10650 3600 10650 4150
-Wire Wire Line
-	10650 4150 10650 4700
+	10650 4150 9750 4150
+Wire Wire Line
+	10650 3400 10650 4700
 Wire Wire Line
 	10300 4700 10300 4150
@@
 Connection ~ 10650 4150
 Wire Wire Line
-	9950 4850 9950 5000
-Wire Wire Line
-	9950 5000 9950 5250
+	9950 4850 9950 5250
 Wire Wire Line
 	9950 4450 9950 4150
@@
 	9950 5650 9950 5900
 Wire Wire Line
-	9950 5900 10300 5900
-Wire Wire Line
-	10300 5900 10650 5900
-Wire Wire Line
-	10300 4900 10300 5900
-Wire Wire Line
-	10300 5900 10300 6000
+	9950 5900 10650 5900
+Wire Wire Line
+	10300 4900 10300 6000
 Wire Wire Line
 	10650 5900 10650 4900
@@
 F 0 "U3" H 7850 4850 60  0000 C CNN
 F 1 "DS7257G" H 8350 4850 60  0000 C CNN
-F 2 "" H 8200 4150 60  0001 C CNN
+F 2 "teensy:SOP-8" H 8200 4150 60  0001 C CNN
 F 3 "" H 8200 4150 60  0001 C CNN
 	1    8200 4150
@@
 	6550 2600 6550 2400
 Wire Wire Line
-	6050 3750 6550 3750
-Wire Wire Line
-	6550 3750 7550 3750
+	6050 3750 7550 3750
 Wire Wire Line
 	6550 3950 6850 3950
@@
 	7250 3950 7550 3950
 Wire Wire Line
-	5450 5300 6000 5300
-Wire Wire Line
-	6000 5300 7100 5300
-Wire Wire Line
-	7100 5300 7400 5300
-Wire Wire Line
-	7400 5300 8200 5300
+	5450 5300 8200 5300
 $Comp
 L RESISTOR_0805 R16
