File: teensy_32_v2/teensy_32_v2.kicad_pcb (KiCad board)
At the start: 2 copper layers, 65 x 56.5 mm, 60 parts, among them J1 277-1667-ND, J2 277-1667-ND, J3 CJ, J4 CJ, J5 CJ, J6 CJ, J7 M20-9980845, J8 M20-9970445, J9 TSW-108-07-G-T, P1 S9200-ND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

Commit message: update footprint for MOSFET
Parts:
- Q1: value STL62P3LLH6 -> STL60P4LLF6
Changed lines of the file:
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@@
 (kicad_pcb (version 4) (host pcbnew 4.0.7-e2-6376~58~ubuntu17.04.1)
   (general
-    (links 158)
+    (links 162)
     (no_connects 0)
     (area 74.949999 59.949999 140.050001 116.550001)
     (thickness 1.6)
     (drawings 87)
-    (tracks 722)
+    (tracks 724)
     (zones 0)
     (modules 60)
@@
   (layers
     (0 F.Cu signal)
-    (31 B.Cu signal)
+    (31 B.Cu signal hide)
     (32 B.Adhes user hide)
     (33 F.Adhes user hide)
@@
   )
   (setup
-    (last_trace_width 0.13)
+    (last_trace_width 0.25)
     (user_trace_width 0.25)
     (user_trace_width 0.45)
@@
       (net 74 /Power/V_SW))
   )
-  (module teensy:POWERFLAT_5x6 (layer F.Cu)
-    (at 87.6935 90.043 180)
-    (attr smd)
-    (fp_text reference Q1 (at -3.2415 -3.4865 270) (layer F.SilkS)
-      (effects (font (size 0.9 0.7) (thickness 0.175)))
-    )
-    (fp_text value STL62P3LLH6 (at 0 -6 180) (layer F.Fab)
-      (effects (font (size 1 1) (thickness 0.15)))
-    )
-    (fp_line (start -2.5 -4.5) (end 2.5 -4.5) (layer F.SilkS) (width 0.15))
-    (fp_line (start 2.5 -4.5) (end 2.5 2) (layer F.SilkS) (width 0.15))
-    (fp_line (start 2.5 2) (end -2.5 2) (layer F.SilkS) (width 0.15))
-    (fp_line (start -2.5 2) (end -2.5 -4.5) (layer F.SilkS) (width 0.15))
-    (pad 3 smd rect (at 0.625 -4.175 180) (size 0.7 0.55) (layers F.Cu F.Paste F.Mask)
-      (net 82 +12V))
-    (pad 3 smd rect (at -0.625 -4.175 180) (size 0.7 0.55) (layers F.Cu F.Paste F.Mask)
-      (net 82 +12V))
-    (pad 3 smd rect (at -1.95 -4.175 180) (size 0.7 0.55) (layers F.Cu F.Paste F.Mask)
-      (net 82 +12V))
-    (pad 2 smd rect (at 1.905 1.525 180) (size 0.635 1.25) (layers F.Cu F.Paste F.Mask)
-      (net 41 "Net-(Q1-Pad2)"))
-    (pad 1 smd rect (at 0.635 1.525 180) (size 0.65 1.25) (layers F.Cu F.Paste F.Mask)
-      (net 78 /Power/VIN))
-    (pad 1 smd rect (at -0.635 1.525 180) (size 0.635 1.25) (layers F.Cu F.Paste F.Mask)
-      (net 78 /Power/VIN))
-    (pad 1 smd rect (at -1.905 1.525 180) (size 0.635 1.25) (layers F.Cu F.Paste F.Mask)
-      (net 78 /Power/VIN))
-    (pad 3 smd rect (at 0 -1.95 180) (size 4.6 3.9) (layers F.Cu F.Paste F.Mask)
-      (net 82 +12V))
-    (pad 3 smd rect (at 1.95 -4.175 180) (size 0.7 0.55) (layers F.Cu F.Paste F.Mask)
-      (net 82 +12V))
-  )
   (module MF_Passives:MF_Passives-R0805 (layer F.Cu)
     (at 92.6465 105.9815 180)
@@
       (net 1 GND))
   )
+  (module teensy:POWERFLAT_5x6 (layer F.Cu)
+    (at 87.6935 90.043 180)
+    (attr smd)
+    (fp_text reference Q1 (at 0 3.5 180) (layer F.SilkS)
+      (effects (font (size 1 1) (thickness 0.15)))
+    )
+    (fp_text value STL60P4LLF6 (at 0 -6 180) (layer F.Fab)
+      (effects (font (size 1 1) (thickness 0.15)))
+    )
+    (fp_line (start -3 1.525) (end -3 1.95) (layer F.SilkS) (width 0.15))
+    (fp_line (start -3.125 1.525) (end -3.125 1.95) (layer F.SilkS) (width 0.15))
+    (fp_line (start -2.875 1.5) (end -2.875 1.975) (layer F.SilkS) (width 0.15))
+    (fp_line (start -2.75 1.5) (end -3.25 1.5) (layer F.SilkS) (width 0.15))
+    (fp_line (start -3.25 1.5) (end -3.25 2) (layer F.SilkS) (width 0.15))
+    (fp_line (start -3.25 2) (end -2.75 2) (layer F.SilkS) (width 0.15))
+    (fp_line (start -2.75 2) (end -2.75 1.5) (layer F.SilkS) (width 0.15))
+    (fp_line (start -2.5 -4.5) (end 2.5 -4.5) (layer F.SilkS) (width 0.15))
+    (fp_line (start 2.5 -4.5) (end 2.5 2) (layer F.SilkS) (width 0.15))
+    (fp_line (start 2.5 2) (end -2.5 2) (layer F.SilkS) (width 0.15))
+    (fp_line (start -2.5 2) (end -2.5 -4.5) (layer F.SilkS) (width 0.15))
+    (pad 3 smd rect (at -2.5 -3.25 180) (size 0.4 0.6) (layers F.Cu F.Paste F.Mask)
+      (net 82 +12V))
+    (pad 3 smd rect (at 2.5 -3.25 180) (size 0.4 0.6) (layers F.Cu F.Paste F.Mask)
+      (net 82 +12V))
+    (pad 3 smd rect (at -2.5 -0.5 180) (size 0.4 0.6) (layers F.Cu F.Paste F.Mask)
+      (net 82 +12V))
+    (pad 3 smd rect (at 0.625 -4.175 180) (size 0.7 0.55) (layers F.Cu F.Paste F.Mask)
+      (net 82 +12V))
+    (pad 3 smd rect (at -0.625 -4.175 180) (size 0.7 0.55) (layers F.Cu F.Paste F.Mask)
+      (net 82 +12V))
+    (pad 3 smd rect (at -1.95 -4.175 180) (size 0.7 0.55) (layers F.Cu F.Paste F.Mask)
+      (net 82 +12V))
+    (pad 2 smd rect (at 1.905 1.525 180) (size 0.635 1.25) (layers F.Cu F.Paste F.Mask)
+      (net 41 "Net-(Q1-Pad2)"))
+    (pad 1 smd rect (at 0.635 1.525 180) (size 0.65 1.25) (layers F.Cu F.Paste F.Mask)
+      (net 78 /Power/VIN))
+    (pad 1 smd rect (at -0.635 1.525 180) (size 0.635 1.25) (layers F.Cu F.Paste F.Mask)
+      (net 78 /Power/VIN))
+    (pad 1 smd rect (at -1.905 1.525 180) (size 0.635 1.25) (layers F.Cu F.Paste F.Mask)
+      (net 78 /Power/VIN))
+    (pad 3 smd rect (at 0 -1.95 180) (size 4.6 3.9) (layers F.Cu F.Paste F.Mask)
+      (net 82 +12V))
+    (pad 3 smd rect (at 1.95 -4.175 180) (size 0.7 0.55) (layers F.Cu F.Paste F.Mask)
+      (net 82 +12V))
+    (pad 3 smd rect (at 2.5 -0.5 180) (size 0.4 0.6) (layers F.Cu F.Paste F.Mask)
+      (net 82 +12V))
+  )
   (gr_text POWER (at 77.5 66.4) (layer F.SilkS)
     (effects (font (size 1.2 0.8) (thickness 0.2)))
@@
   (via (at 132.3086 80.137) (size 0.465) (drill 0.31) (layers F.Cu B.Cu) (net 0))
   (via (at 130.048 80.137) (size 0.465) (drill 0.31) (layers F.Cu B.Cu) (net 0))
+  (segment (start 83.6422 103.4858) (end 85.2932 105.1368) (width 0.25) (layer B.Cu) (net 1))
+  (segment (start 85.2932 105.6132) (end 85.28558 108.35386) (width 0.25) (layer F.Cu) (net 1) (status 800000))
+  (via (at 85.2932 105.6132) (size 0.465) (drill 0.31) (layers F.Cu B.Cu) (net 1))
+  (segment (start 85.2932 105.1368) (end 85.2932 105.6132) (width 0.25) (layer B.Cu) (net 1))
   (segment (start 118.6507 107.3) (end 117.6 107.3) (width 0.25) (layer F.Cu) (net 1))
   (segment (start 117.16 106.86) (end 117.16 103.54) (width 0.25) (layer F.Cu) (net 1))
@@
   (segment (start 101.20122 113.03254) (end 104.2035 113.03254) (width 0.25) (layer F.Cu) (net 1))
   (segment (start 104.2035 113.03254) (end 104.267 112.96904) (width 0.25) (layer F.Cu) (net 1))
-  (segment (start 80.01 97.79) (end 80.01 102.79) (width 0.25) (layer B.Cu) (net 1))
-  (segment (start 80.01 102.79) (end 80.02 102.8) (width 0.25) (layer B.Cu) (net 1))
-  (segment (start 80.02 102.8) (end 83.6 102.8) (width 0.25) (layer B.Cu) (net 1))
-  (via (at 83.6 102.8) (size 0.465) (drill 0.31) (layers F.Cu B.Cu) (net 1))
-  (segment (start 83.6 102.8) (end 85.28558 104.48558) (width 0.25) (layer F.Cu) (net 1))
-  (segment (start 85.28558 104.48558) (end 85.28558 108.35386) (width 0.25) (layer F.Cu) (net 1))
+  (segment (start 80.01 97.79) (end 80.01 103.4758) (width 0.25) (layer B.Cu) (net 1) (status 400000))
+  (segment (start 80.01 103.4758) (end 80.02 103.4858) (width 0.25) (layer B.Cu) (net 1))
+  (segment (start 80.02 103.4858) (end 83.6422 103.4858) (width 0.25) (layer B.Cu) (net 1))
+  (segment (start 83.6422 103.4858) (end 83.6 103.4858) (width 0.25) (layer B.Cu) (net 1))
   (segment (start 114.62 103.54) (end 117.16 103.54) (width 0.7) (layer B.Cu) (net 1))
   (segment (start 112.08 103.54) (end 114.62 103.54) (width 0.7) (layer B.Cu) (net 1))
@@
     (polygon
       (pts
-        (xy 98.2 90.6) (xy 98.2 105.6) (xy 97 105.6) (xy 93.8 102.4) (xy 75.4 102.4)
-        (xy 75.4 89.8) (xy 97.4 89.8)
+        (xy 98.2 90.6) (xy 98.2 105.6) (xy 97 105.6) (xy 93.8508 108.8008) (xy 75.2222 108.8008)
+        (xy 75.1714 89.8) (xy 97.4 89.8)
       )
     )
@@
       )
     )
-  )
-  (zone (net 1) (net_name GND) (layer F.Cu) (hatch edge 0.508)
-    (priority 11)
-    (connect_pads thru_hole_only (clearance 0.2032))
-    (min_thickness 0.1524)
-    (fill yes (arc_segments 16) (thermal_gap 0.3048) (thermal_bridge_width 0.889))
-    (polygon
-      (pts
-        (xy 75 97) (xy 81.6 97) (xy 81.6 104) (xy 75 104)
-      )
-    )

Commit message: make I2C/RPiUART port supply 3V.
Connections:
- J8 pad 5: +5V -> +3V3
- J8 pad 6: +5V -> +3V3
Routing:
- net +3V3: track 55.2 -> 60.6 mm
- net +5V: track 208.3 -> 203.6 mm
- net /T_TX2: track 20.5 -> 21.0 mm, vias 2 -> 1
- net /T_RX3: track 28.4 -> 28.5 mm, vias 3 -> 1
- net (no net): vias 4 -> 5
Other:
- board text added: "+3"

Commit message: tvs/zener protections
Parts:
- added D8: SMAJ16A-E3/61, Diodes_SMD:D_SMA_Standard, B.Cu at (93.5, 94.3)
- added D9: 824500850, Diodes_SMD:D_SMA_Standard, B.Cu at (90.0, 105.8)
- moved C4 0.11 mm to (93.0, 88.5)
Routing:
- net /Power/V_VIN: track 37.4 -> 42.4 mm
- net /Power/VIN: track 45.3 -> 48.2 mm
- net Net-(D9-Pad2): track 27.1 -> 29.4 mm
Other:
- board text added: "2018-01-01"
- board text added: "Teensy Hat for Donkey Car github.com/jwatte/donkey_racing 2018-01-01"
- board text removed: "2017-12-30"
- board text removed: "Teensy Hat for Donkey Car github.com/jwatte/donkey_racing 2017-12-30"
